File: TestBed1/LEDs.kicad_sch (KiCad schematic)
At the start: 22 parts, among them J10 DisplaySegment, U3 TLC5973, U6 TXB0101DBV

Commit message: WIP need layout and reconfiguring
Parts:
- added D10, D8, D9: LED, LED_SMD:LED_Luminus_MP-3030-1100_3.0x3.0mm, symbol Device:LED
Connections:
- net +5V: now also D10.2 (A), D8.2 (A), D9.2 (A)
- net D1: now also D8.1 (K)
- net D2: now also D9.1 (K)
- net D3: now also D10.1 (K)
Other:
- moved on the sheet: C2, R2, TP4, U3

Commit message: Rough Placement and board outline
Parts:
- removed J10: DisplaySegment, X27:DisplayPassthrough, symbol Connector_Generic:Conn_02x02_Counter_Clockwise
- added J7: Conn_01x02_Pin, Connector_PinHeader_1.27mm:PinHeader_1x02_P1.27mm_Vertical, symbol Connector:Conn_01x02_Pin
Connections:
- net +3V3: now also J7.2 (Pin_2)
- net AMB_OUT: now also J7.1 (Pin_1)
Other:
- note added: "Photodetector path i.e. CdS photoresistor"
- moved on the sheet: C11, U7

Commit message: WIP - routing
Connections:
- net D1: now also U3.3 (OUT2); no longer U3.1 (OUT0)
- net D3: now also U3.1 (OUT0); no longer U3.3 (OUT2)
Changed lines of the file:
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@@
-		)
-	)
-	(label "D1"
-		(at 161.29 59.69 0)
-		(fields_autoplaced yes)
-		(effects
-			(font
-				(size 1.27 1.27)
-			)
-			(justify left bottom)
 		)
 	)
@@
 		)
 	)
-	(label "D3"
+	(label "D1"
 		(at 161.29 64.77 0)
 		(fields_autoplaced yes)
@@
 		(fields_autoplaced yes)
 		(effects
+			(font
+				(size 1.27 1.27)
+			)
+			(justify left bottom)
+		)
+	)
+	(label "D3"
+		(at 161.29 59.69 0)
+		(fields_autoplaced yes)
+		(effects
